Commit message: rviz simulation setup

File: dodge_bringup/urdf/dodgebot.xacro (robot description, xacro)
@@ -1,5 +1,5 @@
 <?xml version="1.0"?>
-<robot name="standard" xmlns:xacro="http://www.ros.org/wiki/xacro">
-    <xacro:arg name="is_simulation" default="true" />
+<robot name="dodgebot" xmlns:xacro="http://www.ros.org/wiki/xacro">
+    <xacro:arg name="is_simulation" default="false" />
     <link name="base_footprint"/>
     <link name="base"></link>
@@ -12,5 +12,5 @@
         <origin rpy="0 0 0" xyz="0 0 1" />
         <parent link="base_footprint" />
-        <child link="base_link" />
+        <child link="base" />
     </joint>
     <joint name="yaw_joint" type="fixed">
@@ -24,13 +24,13 @@
         <child link="platform_link" />
     </joint>
-    <joint name="fric_wheel_left_joint" type="continuous">
+    <joint name="fric_wheel_left_joint" type="fixed">
         <origin rpy="0 0 0" xyz="0.1 0.1 0" />
         <parent link="platform_link" />
         <child link="fric_left_wheel" />
     </joint>
-    <joint name="fric_wheel_right_joint" type="continuous">
+    <joint name="fric_wheel_right_joint" type="fixed">
         <origin rpy="0 0 0" xyz="0.1 -0.1 0" />
-        <parent link="base_footprint" />
-        <child link="frick_right_wheel" />
+        <parent link="platform_link" />
+        <child link="fric_right_wheel" />
     </joint>
     <xacro:macro name="shooter_transmission" params="prefix mechanical_reduction motor_id">
@@ -48,5 +48,5 @@
     </xacro:macro>
     <xacro:macro name="gimbal_transmission" params="prefix mechanical_reduction motor_id">
-        <joint name="{prefix}_joint">
+        <joint name="${prefix}_joint">
             <command_interface name="position" />
             <state_interface name="position" />
@@ -86,6 +86,4 @@
         </ros2_control>
     </xacro:unless>
-    <xacro:unless value="$(arg is_simulation)">
-    </xacro:unless>
     <xacro:if value="$(arg is_simulation)">
         <ros2_control name="dji_motors_chassis" type="system">
@@ -106,6 +104,3 @@
         </ros2_control>
     </xacro:if>
-    <xacro:if value="$(arg is_simulation)">
-        <xacro:include filename="$(find metav_description)/urdf/standard/standard.gazebo.xacro" />
-    </xacro:if>
 </robot>

Commit message: stl files added

File: dodge_bringup/urdf/dodgebot.xacro (robot description, xacro)
@@ -4,6 +4,28 @@
     <link name="base_footprint"/>
     <link name="base"></link>
-    <link name="neck_link" />
-    <link name="platform_link" />
+    <link name="neck_link">
+        <visual>
+            <origin xyz="-0.1 -0.15 0.2" rpy="0 1.85 0" />
+            <geometry>
+                <mesh filename="file://$(find dodge_bringup)/meshes/6006yaw.stl"
+                    scale="0.001 0.001 0.001" />
+            </geometry>
+            <material name="silver">
+                <color rgba="0.700 0.700 0.700 1.000" />
+            </material>
+        </visual>
+    </link>
+    <link name="platform_link">
+        <visual>
+            <origin xyz="0 0 0" rpy="0 1.85 0" />
+            <geometry>
+                <mesh filename="file://$(find dodge_bringup)/meshes/gimbal.stl"
+                    scale="0.001 0.001 0.001" />
+            </geometry>
+            <material name="silver">
+                <color rgba="0.700 0.700 0.700 1.000" />
+            </material>
+        </visual>
+    </link>
     <link name="fric_left_wheel" />
     <link name="fric_right_wheel" />

Commit message: dodgebot xacro modificatiomn

File: dodge_bringup/urdf/dodgebot.xacro (robot description, xacro)
@@ -18,5 +18,5 @@
     <link name="platform_link">
         <visual>
-            <origin xyz="0 0 0" rpy="0 1.85 0" />
+            <origin xyz="-0.28 -0.15 0.11" rpy="0 1.85 0" />
             <geometry>
                 <mesh filename="file://$(find dodge_bringup)/meshes/gimbal.stl"
@@ -36,11 +36,23 @@
         <child link="base" />
     </joint>
+    <!-- <joint name="yaw_joint" type="revolute">
+        <origin rpy="0 0 0" xyz="0 0 0" />
+        <limit effort="3." velocity="8.0" lower="-1.5708" upper="1.5708" />
+        <dynamics damping="0.0" friction="0.0" />
+        <safety_controller k_position="100" k_velocity="0.1"
+                soft_lower_limit="0"
+                soft_upper_limit="1000" />
+        <parent link="base" />
+        <child link="neck_link" />
+        <axis xyz="0 1 0" />
+    </joint> -->
     <joint name="yaw_joint" type="fixed">
         <origin rpy="0 0 0" xyz="0 0 0" />
         <parent link="base" />
         <child link="neck_link" />
+        <axis xyz="0 1 0" />
     </joint>
     <joint name="pitch_joint" type="fixed">
-        <origin rpy="0 0 0" xyz="0 0 1" />
+        <origin rpy="0 0 0" xyz="0 0 0.3" />
         <parent link="neck_link" />
         <child link="platform_link" />

Commit message: data calculated

File: dodge_bringup/urdf/dodgebot.xacro (robot description, xacro)
@@ -82,5 +82,5 @@
     </xacro:macro>
     <xacro:macro name="gimbal_transmission" params="prefix mechanical_reduction motor_id">
-        <joint name="${prefix}_joint">
+        <joint name="${prefix}_gimbal_joint">
             <command_interface name="position" />
             <state_interface name="position" />
@@ -109,5 +109,5 @@
             <xacro:shooter_transmission prefix="loader" mechanical_reduction="20.0" motor_id="3" />
         </ros2_control>
-        <!-- <ros2_control name="dm_motros" type="system">
+        <ros2_control name="dm_motros" type="system">
             <hardware>
                 <plugin>meta_hardware/MetaRobotDmMotorNetwork</plugin>
@@ -115,7 +115,7 @@
                 <param name="master_id">0</param>
             </hardware>
-            <xacro:gimbal_transmission prefix="yaw" mechanical_reduction="1.0" motor_id="1" />
-            <xacro:gimbal_transmission prefix="pitch" mechanical_reduction="1.0" motor_id="2" />
-        </ros2_control> -->
+            <xacro:gimbal_transmission prefix="yaw" mechanical_reduction="1.0" motor_id="2" />
+            <xacro:gimbal_transmission prefix="pitch" mechanical_reduction="1.0" motor_id="1" />
+        </ros2_control>
     </xacro:unless>
     <xacro:if value="$(arg is_simulation)">

Commit message: detection overall function complete

File: dodge_bringup/urdf/dodgebot.xacro (robot description, xacro)
@@ -67,4 +67,18 @@
         <parent link="platform_link" />
         <child link="fric_right_wheel" />
+    </joint>
+    <link name="camera_link" />
+    <joint name="camera_joint" type="fixed">
+        <origin xyz="0 0 0" rpy="0 0 0" />
+        <parent link="platform_link" />
+        <child link="camera_link" />
+        <axis xyz="0 0 0" />
+    </joint>
+    <link name="camera_optical_frame" />
+    <joint name="camera_optical_joint" type="fixed">
+        <origin xyz="1 0 0" rpy="${-pi/2} 0 ${-pi/2}" />
+        <!-- <origin xyz="1 0 0" rpy="${pi/2} 0 0" /> -->
+        <parent link="camera_link" />
+        <child link="camera_optical_frame" />
     </joint>
     <xacro:macro name="shooter_transmission" params="prefix mechanical_reduction motor_id">

Commit message: vison enabled; target z position bug encountered.

File: dodge_bringup/urdf/dodgebot.xacro (robot description, xacro)
@@ -47,15 +47,4 @@
         <axis xyz="0 1 0" />
     </joint> -->
-    <joint name="yaw_joint" type="fixed">
-        <origin rpy="0 0 0" xyz="0 0 0" />
-        <parent link="base" />
-        <child link="neck_link" />
-        <axis xyz="0 1 0" />
-    </joint>
-    <joint name="pitch_joint" type="fixed">
-        <origin rpy="0 0 0" xyz="0 0 0.3" />
-        <parent link="neck_link" />
-        <child link="platform_link" />
-    </joint>
     <joint name="fric_wheel_left_joint" type="fixed">
         <origin rpy="0 0 0" xyz="0.1 0.1 0" />
@@ -70,5 +59,5 @@
     <link name="camera_link" />
     <joint name="camera_joint" type="fixed">
-        <origin xyz="0 0 0" rpy="0 0 0" />
+        <origin xyz="0 0 0" rpy="${pi} 0 0" />
         <parent link="platform_link" />
         <child link="camera_link" />
@@ -77,8 +66,22 @@
     <link name="camera_optical_frame" />
     <joint name="camera_optical_joint" type="fixed">
-        <origin xyz="1 0 0" rpy="${-pi/2} 0 ${-pi/2}" />
+        <origin xyz="0.28 0 0.16" rpy="${-pi/2} 0 ${-pi/2}" />
         <!-- <origin xyz="1 0 0" rpy="${pi/2} 0 0" /> -->
         <parent link="camera_link" />
         <child link="camera_optical_frame" />
+    </joint>
+    <joint name="yaw_gimbal_joint" type="continuous">
+            <origin xyz="0 0 0.162" rpy="0 0 0" />
+            <!-- <dynamics damping="0.0" friction="0.1" /> -->
+            <!-- <limit effort="1.2" velocity="31" /> -->
+            <parent link="base" />
+            <child link="neck_link" />
+            <axis xyz="0 0 1" />
+    </joint>
+    <joint name="pitch_gimbal_joint" type="continuous">
+        <origin rpy="${pi} 0 0" xyz="0 0 0.3" />
+        <parent link="neck_link" />
+        <child link="platform_link" />
+        <axis xyz="0 1 0 " />
     </joint>
     <xacro:macro name="shooter_transmission" params="prefix mechanical_reduction motor_id">
@@ -95,5 +98,5 @@
         </joint>
     </xacro:macro>
-    <xacro:macro name="gimbal_transmission" params="prefix mechanical_reduction motor_id">
+    <xacro:macro name="gimbal_transmission" params="prefix mechanical_reduction motor_id offset">
         <joint name="${prefix}_gimbal_joint">
             <command_interface name="position" />
@@ -107,5 +110,5 @@
             <param name="max_vel">30</param>
             <param name="max_effort">10</param>
-            <param name="offset">0.0</param>
+            <param name="offset">${offset}</param>
             <param name="control_mode">mit</param>
             <param name="Kp">30.0</param>
@@ -117,5 +120,5 @@
             <hardware>
                 <plugin>meta_hardware/MetaRobotDjiMotorNetwork</plugin>
-                <param name="can_network_name">can0</param>
+                <param name="can_network_name">can1</param>
             </hardware>
             <xacro:shooter_transmission prefix="fric_wheel_left" mechanical_reduction="-1.0" motor_id="1" />
@@ -126,9 +129,9 @@
             <hardware>
                 <plugin>meta_hardware/MetaRobotDmMotorNetwork</plugin>
-                <param name="can_network_name">can0</param>
+                <param name="can_network_name">can1</param>
                 <param name="master_id">0</param>
             </hardware>
-            <xacro:gimbal_transmission prefix="yaw" mechanical_reduction="1.0" motor_id="1" />
-            <xacro:gimbal_transmission prefix="pitch" mechanical_reduction="1.0" motor_id="2" />
+            <xacro:gimbal_transmission prefix="yaw" mechanical_reduction="1.0" motor_id="1" offset="-0.06"/>
+            <xacro:gimbal_transmission prefix="pitch" mechanical_reduction="1.0" motor_id="2" offset="-1.438"/>
         </ros2_control>
     </xacro:unless>

Commit message: human following first version finished

File: dodge_bringup/urdf/dodgebot.xacro (robot description, xacro)
@@ -98,5 +98,5 @@
         </joint>
     </xacro:macro>
-    <xacro:macro name="gimbal_transmission" params="prefix mechanical_reduction motor_id offset">
+    <xacro:macro name="gimbal_transmission" params="prefix mechanical_reduction motor_id offset mode">
         <joint name="${prefix}_gimbal_joint">
             <command_interface name="position" />
@@ -108,8 +108,8 @@
             <param name="mechanical_reduction">${mechanical_reduction}</param>
             <param name="max_pos">3.141593</param>
-            <param name="max_vel">30</param>
+            <param name="max_vel">0.4</param>
             <param name="max_effort">10</param>
             <param name="offset">${offset}</param>
-            <param name="control_mode">mit</param>
+            <param name="control_mode">${mode}</param>
             <param name="Kp">30.0</param>
             <param name="Kd">0.5</param>
@@ -132,6 +132,6 @@
                 <param name="master_id">0</param>
             </hardware>
-            <xacro:gimbal_transmission prefix="yaw" mechanical_reduction="1.0" motor_id="1" offset="-0.06"/>
-            <xacro:gimbal_transmission prefix="pitch" mechanical_reduction="1.0" motor_id="2" offset="-1.438"/>
+            <xacro:gimbal_transmission prefix="yaw" mechanical_reduction="1.0" motor_id="1" offset="-0.06" mode="mit"/>
+            <xacro:gimbal_transmission prefix="pitch" mechanical_reduction="1.0" motor_id="2" offset="-1.438" mode="mit"/>
         </ros2_control>
     </xacro:unless>
